File: esp32-s3-testboard/esp32-s3-testboard.kicad_pcb (KiCad board)
At the start: 4 copper layers, 50 x 50 mm, 42 parts, among them J1 USB_C_Receptacle_USB2.0_16P, J2 JST_SH_SM04B-SRSS-TB_1x04-1MP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, J4 Pin_02x05, SW2 USER_SW, U1 USBLC6-2SC6, U2 ESP32-S3-WROOM-1, U3 LM1117DT-3.3, U4 Si7020-A20

Commit message: touches
Parts:
- added REF**: KiCad-Logo2_5mm_SilkScreen, Symbol:KiCad-Logo2_5mm_SilkScreen, F.Cu at (125.0, 79.7)
- added REF**: OSHW-Logo_5.7x6mm_SilkScreen, Symbol:OSHW-Logo_5.7x6mm_SilkScreen, F.Cu at (139.0, 54.5)
Other:
- board text added: "Ashen Chathuranga @ktauchathuranga"
- board text added: "ESP32-S3 Tstkit1"
