File: esp32-s3-testboard/esp32-s3-testboard.kicad_sch (KiCad schematic)
At the start: 42 parts, among them J1 USB_C_Receptacle_USB2.0_16P, J2 JST_SH_SM04B-SRSS-TB_1x04-1MP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, J3 Conn_02x03_Odd_Even, J4 Pin_02x05, SW1 RESET, SW2 USER_SW, SW3 BOOT, U1 USBLC6-2SC6, U2 ESP32-S3-WROOM-1, U3 LM1117DT-3.3, U4 Si7021-A20

Commit message: completeddd
Parts:
- removed D5: CLV1L-FKB, LED_SMD:LED_Cree-PLCC4_3.2x2.8mm_CCW, symbol LED:CLV1L-FKB
- removed U4: Si7021-A20, Package_DFN_QFN:DFN-6-1EP_3x3mm_P1mm_EP1.5x2.4mm, symbol Sensor_Humidity:Si7021-A20
- added D5: CLV1L-FKB, oddibits:LED_Cree-PLCC4_3.2x2.8mm_CCW, symbol oddibits:CLV1L-FKB
- added U4: Si7020-A20, oddibits:DFN-6-1EP_3x3mm_P1mm_EP1.5x2.4mm, symbol oddibits:Si7020-A20
- D1: footprint Diode_THT:D_DO-41_SOD81_P10.16mm_Horizontal -> Diode_SMD:D_SOD-123
- U3: footprint Package_TO_SOT_SMD:SOT-223 -> Package_TO_SOT_SMD:SOT-223-3_TabPin2
Connections:
- net +3V3: now also D5.1 (A), U4.5 (VDD)
- net D+: now also U1.3 (I/O2); no longer U1.1 (I/O1)
- net D-: now also U1.1 (I/O1); no longer U1.3 (I/O2)
- net GND: now also U4.2 (GND)
- net SCL: now also U4.6 (SCL)
- net SDA: now also U4.1 (SDA)
- net USB_D+: now also U1.4 (I/O2); no longer U1.6 (I/O1)
- net USB_D-: now also U1.6 (I/O1); no longer U1.4 (I/O2)
- net at R9.1: now also D5.2 (RK)
- net at R10.1: now also D5.3 (GK)
- net at R11.1: now also D5.4 (BK)
Changed lines of the file:
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@@
 	)
 	(label "USB_D-"
-		(at 91.44 50.8 0)
+		(at 91.44 48.26 0)
 		(effects
 			(font
@@
 	)
 	(label "D-"
-		(at 68.58 50.8 0)
+		(at 68.58 48.26 0)
 		(effects
 			(font
@@
 	)
 	(label "D+"
-		(at 68.58 48.26 0)
+		(at 68.58 50.8 0)
 		(effects
 			(font
@@
 	)
 	(label "USB_D+"
-		(at 91.44 48.26 0)
+		(at 91.44 50.8 0)
 		(effects
 			(font
@@
 	)
 	(symbol
+		(lib_id "oddibits:CLV1L-FKB")
+		(at 27.94 161.29 0)
+		(mirror y)
+		(unit 1)
+		(exclude_from_sim no)
+		(in_bom yes)
+		(on_board yes)
+		(dnp no)
+		(property "Reference" "D5"
+			(at 27.94 147.32 0)
+			(effects
+				(font
+					(size 1.27 1.27)
+				)
+			)
+		)
+		(property "Value" "CLV1L-FKB"
+			(at 27.94 149.86 0)
+			(effects
+				(font
+					(size 1.27 1.27)
+				)
+			)
+		)
+		(property "Footprint" "oddibits:LED_Cree-PLCC4_3.2x2.8mm_CCW"
+			(at 27.94 162.56 0)
+			(effects
+				(font
+					(size 1.27 1.27)
+				)
+				(hide yes)
+			)
+		)
+		(property "Datasheet" "http://www.cree.com/led-components/media/documents/CLV1L-FKB-1238.pdf"
+			(at 27.94 162.56 0)
+			(effects
+				(font
+					(size 1.27 1.27)
+				)
+				(hide yes)
+			)
+		)
+		(property "Description" "Cree PLCC4 3 in 1 SMD LED"
+			(at 27.94 161.29 0)
+			(effects
+				(font
+					(size 1.27 1.27)
+				)
+				(hide yes)
+			)
+		)
+		(pin "3"
+		)
+		(pin "2"
+		)
+		(pin "4"
+		)
+		(pin "1"
+		)
+		(instances
+			(project ""
+				(path "/a7f6de19-e097-4448-b7dc-f3b51ffbf1c5"
+					(reference "D5")
+					(unit 1)
+				)
+			)
+		)
+	)
+	(symbol
 		(lib_id "Device:C_Small")
 		(at 92.71 36.83 0)
@@
 	)
 	(symbol
+		(lib_id "oddibits:Si7020-A20")
+		(at 132.08 180.34 0)
+		(unit 1)
+		(exclude_from_sim no)
+		(in_bom yes)
+		(on_board yes)
+		(dnp no)
+		(fields_autoplaced yes)
+		(property "Reference" "U4"
+			(at 143.51 179.0699 0)
+			(effects
+				(font
+					(size 1.27 1.27)
+				)
+				(justify left)
+			)
+		)
+		(property "Value" "Si7020-A20"
+			(at 143.51 181.6099 0)
+			(effects
+				(font
+					(size 1.27 1.27)
+				)
+				(justify left)
+			)
+		)
+		(property "Footprint" "oddibits:DFN-6-1EP_3x3mm_P1mm_EP1.5x2.4mm"
+			(at 132.08 190.5 0)
+			(effects
+				(font
+					(size 1.27 1.27)
+				)
+				(hide yes)
+			)
+		)
+		(property "Datasheet" "https://www.silabs.com/documents/public/data-sheets/Si7020-A20.pdf"
+			(at 127 172.72 0)
+			(effects
+				(font
+					(size 1.27 1.27)
+				)
+				(hide yes)
+			)
+		)
+		(property "Description" "I2C Humidity and Temperature Sensor, DFN-6"
+			(at 132.08 180.34 0)
+			(effects
+				(font
+					(size 1.27 1.27)
+				)
+				(hide yes)
+			)
+		)
+		(pin "1"
+		)
+		(pin "5"
+		)
+		(pin "2"
+		)
+		(pin "6"
+		)
+		(pin "4"
+		)
+		(pin "7"
+		)
+		(pin "3"
+		)
+		(instances
+			(project ""
+				(path "/a7f6de19-e097-4448-b7dc-f3b51ffbf1c5"
+					(reference "U4")
+					(unit 1)
+				)
+			)
+		)
+	)
+	(symbol
 		(lib_id "oddibits:JST_SH_SM04B-SRSS-TB_1x04-1MP_P1.00mm_Horizontal")
 		(at 57.15 133.35 0)
@@
 			)
 		)
-		(property "Footprint" "Diode_THT:D_DO-41_SOD81_P10.16mm_Horizontal"
+		(property "Footprint" "Diode_SMD:D_SOD-123"
 			(at 88.9 17.145 0)
 			(effects
@@
 	)
 	(symbol
-		(lib_id "Sensor_Humidity:Si7021-A20")
-		(at 132.08 180.34 0)
-		(unit 1)
-		(exclude_from_sim no)
-		(in_bom yes)
-		(on_board yes)
-		(dnp no)
-		(fields_autoplaced yes)
-		(property "Reference" "U4"
-			(at 143.51 179.0699 0)
-			(effects
-				(font
-					(size 1.27 1.27)
-				)
-				(justify left)
-			)
-		)
-		(property "Value" "Si7021-A20"
-			(at 143.51 181.6099 0)
-			(effects
-				(font
-					(size 1.27 1.27)
-				)
-				(justify left)
-			)
-		)
-		(property "Footprint" "Package_DFN_QFN:DFN-6-1EP_3x3mm_P1mm_EP1.5x2.4mm"
-			(at 132.08 190.5 0)
-			(effects
-				(font
-					(size 1.27 1.27)
-				)
-				(hide yes)
-			)
-		)
-		(property "Datasheet" "https://www.silabs.com/documents/public/data-sheets/Si7021-A20.pdf"
-			(at 127 172.72 0)
-			(effects
-				(font
-					(size 1.27 1.27)
-				)
-				(hide yes)
-			)
-		)
-		(property "Description" "I2C Humidity and Temperature Sensor, DFN-6"
-			(at 132.08 180.34 0)
-			(effects
-				(font
-					(size 1.27 1.27)
-				)
-				(hide yes)
-			)
-		)
-		(pin "3"
-		)
-		(pin "7"
-		)
-		(pin "1"
-		)
-		(pin "2"
-		)
-		(pin "6"
-		)
-		(pin "4"
-		)
-		(pin "5"
-		)
-		(instances
-			(project ""
-				(path "/a7f6de19-e097-4448-b7dc-f3b51ffbf1c5"
-					(reference "U4")
-					(unit 1)
-				)
-			)
-		)
-	)
-	(symbol
 		(lib_id "power:GND")
 		(at 91.44 123.19 0)
@@
 			)
 		)
-		(property "Footprint" "Package_TO_SOT_SMD:SOT-223"
+		(property "Footprint" "Package_TO_SOT_SMD:SOT-223-3_TabPin2"
 			(at 34.29 91.44 0)
 			(effects
@@
 					(unit 1)
 				)
-			)
-		)
-	)
-	(symbol
-		(lib_id "LED:CLV1L-FKB")
-		(at 27.94 161.29 0)
-		(mirror y)
-		(unit 1)
-		(exclude_from_sim no)
-		(in_bom yes)
-		(on_board yes)
-		(dnp no)
-		(property "Reference" "D5"
-			(at 27.94 148.59 0)
-			(effects
-				(font
-					(size 1.27 1.27)
-				)
-			)
-		)
-		(property "Value" "CLV1L-FKB"
-			(at 27.94 151.13 0)
-			(effects
-				(font
-					(size 1.27 1.27)
-				)
-			)
-		)
-		(property "Footprint" "LED_SMD:LED_Cree-PLCC4_3.2x2.8mm_CCW"
-			(at 27.94 162.56 0)
-			(effects
-				(font
-					(size 1.27 1.27)
-				)
-				(hide yes)
-			)
-		)
-		(property "Datasheet" "http://www.cree.com/led-components/media/documents/CLV1L-FKB-1238.pdf"
-			(at 27.94 162.56 0)
-			(effects
-				(font
-					(size 1.27 1.27)
-				)
-				(hide yes)
-			)
-		)
-		(property "Description" "Cree PLCC4 3 in 1 SMD LED"
-			(at 27.94 161.29 0)
-			(effects
-				(font
-					(size 1.27 1.27)
-				)
-				(hide yes)
-			)
-		)
-		(pin "1"
-		)
-		(pin "4"
-		)
-		(pin "3"
-		)
-		(pin "2"
-		)
-		(instances
-			(project ""
-				(path "/a7f6de19-e097-4448-b7dc-f3b51ffbf1c5"
-					(reference "D5")
-					(unit 1)
-				)

Commit message: touches
Other:
- moved on the sheet: C1, C2, C3, C4, C5, C6, C7, C8, D1, D2, D3, D4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
